Commit message: urdfぶっ壊れた。ねむいからねる

File: src/robot26a_urdf/urdf/ros26a_urdf.xacro (robot description, xacro)
@@ -1,235 +1,224 @@
-<?xml version="1.0" ?>
-<robot name="ros26a_urdf" xmlns:xacro="http://www.ros.org/wiki/xacro">
+<?xml version='1.0' encoding='utf-8'?>
+<robot xmlns:xacro="http://www.ros.org/wiki/xacro" name="ros26a_urdf">
 <xacro:include filename="$(find robot26a_urdf)/urdf/materials.xacro" />
-<xacro:include filename="$(find robot26a_urdf)/urdf/ros26a_urdf.ros2control" />
+<xacro:include filename="$(find robot26a_urdf)/urdf/ros26a_urdf.ros2control.xml" />
 <xacro:include filename="$(find robot26a_urdf)/urdf/ros26a_urdf.gazebo" />
 <link name="base_link">
   <inertial>
-    <origin xyz="-2.419230684947819e-05 -0.02126179221935003 0.10065551791673599" rpy="0 0 0"/>
-    <mass value="4.390871082692601"/>
-    <inertia ixx="0.390977" iyy="0.367331" izz="0.702941" ixy="6e-06" iyz="0.018528" ixz="2e-06"/>
-  </inertial>
-  <visual>
-    <origin xyz="0 0 0" rpy="0 0 0"/>
-    <geometry>
-      <mesh filename="file://$(find robot26a_urdf)/meshes/base_link.stl" scale="0.001 0.001 0.001"/>
-    </geometry>
-    <material name="silver"/>
-  </visual>
-  <collision>
-    <origin xyz="0 0 0" rpy="0 0 0"/>
-    <geometry>
-      <mesh filename="file://$(find robot26a_urdf)/meshes/base_link.stl" scale="0.001 0.001 0.001"/>
-    </geometry>
-  </collision>
-</link>
-<link name="wheel_rear_right_link">
-  <inertial>
-    <origin xyz="0.033324758909945684 0.03336765433449884 8.127027229271055e-06" rpy="0 0 0"/>
-    <mass value="2.8236842197299814"/>
-    <inertia ixx="0.006412" iyy="0.006411" izz="0.004583" ixy="0.001829" iyz="1e-06" ixz="1e-06"/>
-  </inertial>
-  <visual>
-    <origin xyz="0.383252 0.383252 -0.076" rpy="0 0 0"/>
-    <geometry>
-      <mesh filename="file://$(find robot26a_urdf)/meshes/wheel_rear_right_link.stl" scale="0.001 0.001 0.001"/>
-    </geometry>
-    <material name="silver"/>
-  </visual>
-  <collision>
-    <origin xyz="0.383252 0.383252 -0.076" rpy="0 0 0"/>
-    <geometry>
-      <mesh filename="file://$(find robot26a_urdf)/meshes/wheel_rear_right_link.stl" scale="0.001 0.001 0.001"/>
-    </geometry>
-  </collision>
-</link>
-<link name="wheel_front_right_link">
-  <inertial>
-    <origin xyz="-0.033351953298285275 0.033340459946157475 -3.033164558431667e-05" rpy="0 0 0"/>
-    <mass value="2.8236842197299814"/>
-    <inertia ixx="0.006413" iyy="0.00641" izz="0.004583" ixy="-0.001828" iyz="0.0" ixz="-0.0"/>
-  </inertial>
-  <visual>
-    <origin xyz="-0.383252 0.383252 -0.076" rpy="0 0 0"/>
-    <geometry>
-      <mesh filename="file://$(find robot26a_urdf)/meshes/wheel_front_right_link.stl" scale="0.001 0.001 0.001"/>
-    </geometry>
-    <material name="silver"/>
-  </visual>
-  <collision>
-    <origin xyz="-0.383252 0.383252 -0.076" rpy="0 0 0"/>
-    <geometry>
-      <mesh filename="file://$(find robot26a_urdf)/meshes/wheel_front_right_link.stl" scale="0.001 0.001 0.001"/>
-    </geometry>
-  </collision>
-</link>
-<link name="wheel_front_left_link">
-  <inertial>
-    <origin xyz="-0.03336765540973269 -0.033324760516337704 -8.12736003742709e-06" rpy="0 0 0"/>
-    <mass value="2.823684325023845"/>
-    <inertia ixx="0.006411" iyy="0.006412" izz="0.004583" ixy="0.001829" iyz="1e-06" ixz="1e-06"/>
-  </inertial>
-  <visual>
-    <origin xyz="-0.383252 -0.383252 -0.076" rpy="0 0 0"/>
-    <geometry>
-      <mesh filename="file://$(find robot26a_urdf)/meshes/wheel_front_left_link.stl" scale="0.001 0.001 0.001"/>
-    </geometry>
-    <material name="silver"/>
-  </visual>
-  <collision>
-    <origin xyz="-0.383252 -0.383252 -0.076" rpy="0 0 0"/>
-    <geometry>
-      <mesh filename="file://$(find robot26a_urdf)/meshes/wheel_front_left_link.stl" scale="0.001 0.001 0.001"/>
-    </geometry>
-  </collision>
-</link>
-<link name="wheel_rear_left_link">
-  <inertial>
-    <origin xyz="0.03332476051633948 -0.03336765540973591 -8.127360037579745e-06" rpy="0 0 0"/>
-    <mass value="2.823684325023845"/>
-    <inertia ixx="0.006412" iyy="0.006411" izz="0.004583" ixy="-0.001829" iyz="1e-06" ixz="-1e-06"/>
-  </inertial>
-  <visual>
-    <origin xyz="0.383252 -0.383252 -0.076" rpy="0 0 0"/>
-    <geometry>
-      <mesh filename="file://$(find robot26a_urdf)/meshes/wheel_rear_left_link.stl" scale="0.001 0.001 0.001"/>
-    </geometry>
-    <material name="silver"/>
-  </visual>
-  <collision>
-    <origin xyz="0.383252 -0.383252 -0.076" rpy="0 0 0"/>
-    <geometry>
-      <mesh filename="file://$(find robot26a_urdf)/meshes/wheel_rear_left_link.stl" scale="0.001 0.001 0.001"/>
-    </geometry>
-  </collision>
-</link>
-<link name="lidar_link">
-  <inertial>
-    <origin xyz="-0.08000446122505181 0.04106120302884397 -0.010858053646773336" rpy="0 0 0"/>
-    <mass value="0.350138445908399"/>
-    <inertia ixx="0.000308" iyy="0.000617" izz="0.00089" ixy="-0.0" iyz="-0.0" ixz="0.0"/>
-  </inertial>
-  <visual>
-    <origin xyz="-0.08 0.374382 -0.433095" rpy="0 0 0"/>
-    <geometry>
-      <mesh filename="file://$(find robot26a_urdf)/meshes/lidar_link.stl" scale="0.001 0.001 0.001"/>
-    </geometry>
-    <material name="silver"/>
-  </visual>
-  <collision>
-    <origin xyz="-0.08 0.374382 -0.433095" rpy="0 0 0"/>
-    <geometry>
-      <mesh filename="file://$(find robot26a_urdf)/meshes/lidar_link.stl" scale="0.001 0.001 0.001"/>
-    </geometry>
-  </collision>
-</link>
-<link name="camera_link">
-  <inertial>
-    <origin xyz="-0.015463046523140393 0.010481077086632706 0.0167332636074774" rpy="0 0 0"/>
-    <mass value="0.06383766089551529"/>
-    <inertia ixx="1.4e-05" iyy="4.7e-05" izz="4.1e-05" ixy="1e-06" iyz="-1e-06" ixz="0.0"/>
-  </inertial>
-  <visual>
-    <origin xyz="-0.015 0.250446 -0.4402" rpy="0 0 0"/>
-    <geometry>
-      <mesh filename="file://$(find robot26a_urdf)/meshes/camera_link.stl" scale="0.001 0.001 0.001"/>
-    </geometry>
-    <material name="silver"/>
-  </visual>
-  <collision>
-    <origin xyz="-0.015 0.250446 -0.4402" rpy="0 0 0"/>
-    <geometry>
-      <mesh filename="file://$(find robot26a_urdf)/meshes/camera_link.stl" scale="0.001 0.001 0.001"/>
-    </geometry>
-  </collision>
-</link>
-<link name="camera_body_link">
-  <inertial>
-    <origin xyz="-0.029749880192293236 0.009806199358828122 1.596729986563794e-07" rpy="0 0 0"/>
-    <mass value="0.017157190826827023"/>
-    <inertia ixx="1e-06" iyy="1.4e-05" izz="1.5e-05" ixy="-0.0" iyz="-0.0" ixz="-0.0"/>
-  </inertial>
-  <visual>
-    <origin xyz="-0.02975 0.251646 -0.4612" rpy="0 0 0"/>
-    <geometry>
-      <mesh filename="file://$(find robot26a_urdf)/meshes/camera_body_link.stl" scale="0.001 0.001 0.001"/>
-    </geometry>
-    <material name="silver"/>
-  </visual>
-  <collision>
-    <origin xyz="-0.02975 0.251646 -0.4612" rpy="0 0 0"/>
-    <geometry>
-      <mesh filename="file://$(find robot26a_urdf)/meshes/camera_body_link.stl" scale="0.001 0.001 0.001"/>
-    </geometry>
-  </collision>
-</link>
-<link name="lidar_head_link">
-  <inertial>
-    <origin xyz="9.354544219402101e-06 -6.517181017173801e-05 -0.016167762462367286" rpy="0 0 0"/>
-    <mass value="0.6884110896982916"/>
-    <inertia ixx="0.000306" iyy="0.000194" izz="0.000371" ixy="7e-06" iyz="-0.0" ixz="0.0"/>
-  </inertial>
-  <visual>
-    <origin xyz="-0.0 0.333335 -0.394095" rpy="0 0 0"/>
-    <geometry>
-      <mesh filename="file://$(find robot26a_urdf)/meshes/lidar_head_link.stl" scale="0.001 0.001 0.001"/>
-    </geometry>
-    <material name="silver"/>
-  </visual>
-  <collision>
-    <origin xyz="-0.0 0.333335 -0.394095" rpy="0 0 0"/>
-    <geometry>
-      <mesh filename="file://$(find robot26a_urdf)/meshes/lidar_head_link.stl" scale="0.001 0.001 0.001"/>
-    </geometry>
+    <origin xyz="-2.4286184067020517e-05 -0.021344258350690065 0.10100713035152749" rpy="0 0 0" />
+    <mass value="4.373906465543717" />
+    <inertia ixx="0.390828" iyy="0.36719" izz="0.702933" ixy="6e-06" iyz="0.018495" ixz="2e-06" />
+  </inertial>
+  <visual>
+    <origin xyz="0 0 0" rpy="0 0 0" />
+    <geometry>
+      <mesh filename="file://$(find robot26a_urdf)/meshes/base_link.stl" scale="0.001 0.001 0.001" />
+    </geometry>
+    <material name="silver" />
+  </visual>
+  <collision>
+    <origin xyz="0 0 0.1" rpy="0 0 0" />
+    <geometry>
+      <box size="0.7 0.7 0.2" /></geometry>
+  </collision>
+</link>
+<link name="omni_2_1">
+  <inertial>
+    <origin xyz="0.033324758909945684 0.03336765433449884 8.127027229271055e-06" rpy="0 0 0" />
+    <mass value="2.8236842197299814" />
+    <inertia ixx="0.006412" iyy="0.006411" izz="0.004583" ixy="0.001829" iyz="1e-06" ixz="1e-06" />
+  </inertial>
+  <visual>
+    <origin xyz="0.383252 0.383252 -0.076" rpy="0 0 0" />
+    <geometry>
+      <mesh filename="file://$(find robot26a_urdf)/meshes/omni_2_1.stl" scale="0.001 0.001 0.001" />
+    </geometry>
+    <material name="silver" />
+  </visual>
+  <collision>
+    <origin xyz="0 0 0" rpy="0 0 0" />
+    <geometry>
+      <sphere radius="0.05" /></geometry>
+  </collision>
+</link>
+<link name="omni_1_1">
+  <inertial>
+    <origin xyz="-0.033351953298285275 0.033340459946157475 -3.033164558431667e-05" rpy="0 0 0" />
+    <mass value="2.8236842197299814" />
+    <inertia ixx="0.006413" iyy="0.00641" izz="0.004583" ixy="-0.001828" iyz="0.0" ixz="-0.0" />
+  </inertial>
+  <visual>
+    <origin xyz="-0.383252 0.383252 -0.076" rpy="0 0 0" />
+    <geometry>
+      <mesh filename="file://$(find robot26a_urdf)/meshes/omni_1_1.stl" scale="0.001 0.001 0.001" />
+    </geometry>
+    <material name="silver" />
+  </visual>
+  <collision>
+    <origin xyz="0 0 0" rpy="0 0 0" />
+    <geometry>
+      <sphere radius="0.05" /></geometry>
+  </collision>
+</link>
+<link name="omni_4_1">
+  <inertial>
+    <origin xyz="-0.03336765540973269 -0.033324760516337704 -8.12736003742709e-06" rpy="0 0 0" />
+    <mass value="2.823684325023845" />
+    <inertia ixx="0.006411" iyy="0.006412" izz="0.004583" ixy="0.001829" iyz="1e-06" ixz="1e-06" />
+  </inertial>
+  <visual>
+    <origin xyz="-0.383252 -0.383252 -0.076" rpy="0 0 0" />
+    <geometry>
+      <mesh filename="file://$(find robot26a_urdf)/meshes/omni_4_1.stl" scale="0.001 0.001 0.001" />
+    </geometry>
+    <material name="silver" />
+  </visual>
+  <collision>
+    <origin xyz="0 0 0" rpy="0 0 0" />
+    <geometry>
+      <sphere radius="0.05" /></geometry>
+  </collision>
+</link>
+<link name="omni_3_1">
+  <inertial>
+    <origin xyz="0.03332476051633948 -0.03336765540973591 -8.127360037579745e-06" rpy="0 0 0" />
+    <mass value="2.823684325023845" />
+    <inertia ixx="0.006412" iyy="0.006411" izz="0.004583" ixy="-0.001829" iyz="1e-06" ixz="-1e-06" />
+  </inertial>
+  <visual>
+    <origin xyz="0.383252 -0.383252 -0.076" rpy="0 0 0" />
+    <geometry>
+      <mesh filename="file://$(find robot26a_urdf)/meshes/omni_3_1.stl" scale="0.001 0.001 0.001" />
+    </geometry>
+    <material name="silver" />
+  </visual>
+  <collision>
+    <origin xyz="0 0 0" rpy="0 0 0" />
+    <geometry>
+      <sphere radius="0.05" /></geometry>
+  </collision>
+</link>
+<link name="r_lidar_1">
+  <inertial>
+    <origin xyz="-0.08000446122505181 0.04106120302884397 -0.010858053646773336" rpy="0 0 0" />
+    <mass value="0.350138445908399" />
+    <inertia ixx="0.000308" iyy="0.000617" izz="0.00089" ixy="-0.0" iyz="-0.0" ixz="0.0" />
+  </inertial>
+  <visual>
+    <origin xyz="-0.08 0.374382 -0.433095" rpy="0 0 0" />
+    <geometry>
+      <mesh filename="file://$(find robot26a_urdf)/meshes/r_lidar_1.stl" scale="0.001 0.001 0.001" />
+    </geometry>
+    <material name="silver" />
+  </visual>
+  <collision>
+    <origin xyz="0 0 0" rpy="0 0 0" />
+    <geometry>
+      <box size="0.05 0.05 0.05" /></geometry>
+  </collision>
+</link>
+<link name="r_cam_1">
+  <inertial>
+    <origin xyz="-0.015463046523140393 0.010481077086632706 0.0167332636074774" rpy="0 0 0" />
+    <mass value="0.06383766089551529" />
+    <inertia ixx="1.4e-05" iyy="4.7e-05" izz="4.1e-05" ixy="1e-06" iyz="-1e-06" ixz="0.0" />
+  </inertial>
+  <visual>
+    <origin xyz="-0.015 0.250446 -0.4402" rpy="0 0 0" />
+    <geometry>
+      <mesh filename="file://$(find robot26a_urdf)/meshes/r_cam_1.stl" scale="0.001 0.001 0.001" />
+    </geometry>
+    <material name="silver" />
+  </visual>
+  <collision>
+    <origin xyz="0 0 0" rpy="0 0 0" />
+    <geometry>
+      <box size="0.05 0.05 0.05" /></geometry>
+  </collision>
+</link>
+<link name="r_cam_body_1">
+  <inertial>
+    <origin xyz="-0.029749880192293236 0.009806199358828122 1.596729986563794e-07" rpy="0 0 0" />
+    <mass value="0.017157190826827023" />
+    <inertia ixx="1e-06" iyy="1.4e-05" izz="1.5e-05" ixy="-0.0" iyz="-0.0" ixz="-0.0" />
+  </inertial>
+  <visual>
+    <origin xyz="-0.02975 0.251646 -0.4612" rpy="0 0 0" />
+    <geometry>
+      <mesh filename="file://$(find robot26a_urdf)/meshes/r_cam_body_1.stl" scale="0.001 0.001 0.001" />
+    </geometry>
+    <material name="silver" />
+  </visual>
+  <collision>
+    <origin xyz="0 0 0" rpy="0 0 0" />
+    <geometry>
+      <box size="0.05 0.05 0.05" /></geometry>
+  </collision>
+</link>
+<link name="r_lidar_head_1">
+  <inertial>
+    <origin xyz="9.354544219402101e-06 -6.517181017173801e-05 -0.016167762462367286" rpy="0 0 0" />
+    <mass value="0.6884110896982916" />
+    <inertia ixx="0.000306" iyy="0.000194" izz="0.000371" ixy="7e-06" iyz="-0.0" ixz="0.0" />
+  </inertial>
+  <visual>
+    <origin xyz="-0.0 0.333335 -0.394095" rpy="0 0 0" />
+    <geometry>
+      <mesh filename="file://$(find robot26a_urdf)/meshes/r_lidar_head_1.stl" scale="0.001 0.001 0.001" />
+    </geometry>
+    <material name="silver" />
+  </visual>
+  <collision>
+    <origin xyz="0 0 0" rpy="0 0 0" />
+    <geometry>
+      <box size="0.05 0.05 0.05" /></geometry>
   </collision>
 </link>
 <joint name="wheel_rear_right_joint" type="continuous">
-  <origin xyz="-0.383252 -0.383252 0.076" rpy="0 0 0"/>
-  <parent link="base_link"/>
-  <child link="wheel_rear_right_link"/>
-  <axis xyz="0.707107 0.707107 -0.0"/>
+  <origin xyz="-0.383252 -0.383252 0.076" rpy="0 0 0" />
+  <parent link="base_link" />
+  <child link="omni_2_1" />
+  <axis xyz="0.707107 0.707107 -0.0" />
 </joint>
 <joint name="wheel_front_right_joint" type="continuous">
-  <origin xyz="0.383252 -0.383252 0.076" rpy="0 0 0"/>
-  <parent link="base_link"/>
-  <child link="wheel_front_right_link"/>
-  <axis xyz="-0.707107 0.707107 -0.0"/>
+  <origin xyz="0.383252 -0.383252 0.076" rpy="0 0 0" />
+  <parent link="base_link" />
+  <child link="omni_1_1" />
+  <axis xyz="-0.707107 0.707107 -0.0" />
 </joint>
 <joint name="wheel_front_left_joint" type="continuous">
-  <origin xyz="0.383252 0.383252 0.076" rpy="0 0 0"/>
-  <parent link="base_link"/>
-  <child link="wheel_front_left_link"/>
-  <axis xyz="-0.707107 -0.707107 0.0"/>
+  <origin xyz="0.383252 0.383252 0.076" rpy="0 0 0" />
+  <parent link="base_link" />
+  <child link="omni_4_1" />
+  <axis xyz="-0.707107 -0.707107 0.0" />
 </joint>
 <joint name="wheel_rear_left_joint" type="continuous">
-  <origin xyz="-0.383252 0.383252 0.076" rpy="0 0 0"/>
-  <parent link="base_link"/>
-  <child link="wheel_rear_left_link"/>
-  <axis xyz="0.707107 -0.707107 0.0"/>
-</joint>
-<joint name="lidar_joint" type="revolute">
-  <origin xyz="0.08 -0.374382 0.433095" rpy="0 0 0"/>
-  <parent link="base_link"/>
-  <child link="lidar_link"/>
-  <axis xyz="-1.0 0.0 0.0"/>
-  <limit lower="0.52359877" upper="0.52359877" effort="100.0" velocity="0.0"/>
-</joint>
-<joint name="camera_joint" type="revolute">
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