Commit message: めっちゃうまく行ったurdf - 2dlidar設置。

File: src/r26a_urdf/r26a_urdf.xacro (robot description, xacro)
@@ -1,11 +1,9 @@
 <?xml version="1.0"?>
 <robot name="r26a_urdf" xmlns:xacro="http://www.ros.org/wiki/xacro">
-  <xacro:include filename="$(find r26a_urdf)/urdf/materials.xacro" />
-  <xacro:include filename="$(find r26a_urdf)/urdf/r26a_urdf.ros2control" />
-  <xacro:include filename="$(find r26a_urdf)/urdf/r26a_urdf.gazebo" />
-  <link name="dummy_link" />
+  <xacro:include filename="materials.xacro" />
+  <link name="dummy"/>
   <joint name="dummy_joint" type="fixed">
-    <parent link="dummy_link" />
-    <child link="base_link" />
+    <parent link="dummy"/>
+    <child link="base_link"/>
   </joint>
   <link name="base_link">
@@ -18,5 +16,6 @@
       <origin xyz="0 0 0" rpy="0 0 0" />
       <geometry>
-        <mesh filename="package://r26a_urdf/meshes/base_link.stl" scale="0.001 0.001 0.001" />
+        <mesh filename="file://$(find r26a_urdf)/meshes/base_link.stl"
+          scale="0.001 0.001 0.001" />
       </geometry>
       <material name="silver" />
@@ -25,5 +24,6 @@
       <origin xyz="0 0 0" rpy="0 0 0" />
       <geometry>
-        <mesh filename="package://r26a_urdf/meshes/base_link.stl" scale="0.001 0.001 0.001" />
+        <mesh filename="file://$(find r26a_urdf)/meshes/base_link.stl"
+          scale="0.001 0.001 0.001" />
       </geometry>
     </collision>
@@ -38,12 +38,14 @@
       <origin xyz="0.383252 0.383252 -0.076" rpy="0 0 0" />
       <geometry>
-        <mesh filename="package://r26a_urdf/meshes/omni_2_1.stl" scale="0.001 0.001 0.001" />
-      </geometry>
-      <material name="silver" />
-    </visual>
-    <collision>
-      <origin xyz="0.03335 0.03335 0" rpy="0 0 0" />
-      <geometry>
-        <sphere radius="0.076" />
+        <mesh filename="file://$(find r26a_urdf)/meshes/omni_2_1.stl"
+          scale="0.001 0.001 0.001" />
+      </geometry>
+      <material name="silver" />
+    </visual>
+    <collision>
+      <origin xyz="0.383252 0.383252 -0.076" rpy="0 0 0" />
+      <geometry>
+        <mesh filename="file://$(find r26a_urdf)/meshes/omni_2_1.stl"
+          scale="0.001 0.001 0.001" />
       </geometry>
     </collision>
@@ -58,12 +60,14 @@
       <origin xyz="-0.383252 0.383252 -0.076" rpy="0 0 0" />
       <geometry>
-        <mesh filename="package://r26a_urdf/meshes/omni_1_1.stl" scale="0.001 0.001 0.001" />
-      </geometry>
-      <material name="silver" />
-    </visual>
-    <collision>
-      <origin xyz="-0.03335 0.03335 0" rpy="0 0 0" />
-      <geometry>
-        <sphere radius="0.076" />
+        <mesh filename="file://$(find r26a_urdf)/meshes/omni_1_1.stl"
+          scale="0.001 0.001 0.001" />
+      </geometry>
+      <material name="silver" />
+    </visual>
+    <collision>
+      <origin xyz="-0.383252 0.383252 -0.076" rpy="0 0 0" />
+      <geometry>
+        <mesh filename="file://$(find r26a_urdf)/meshes/omni_1_1.stl"
+          scale="0.001 0.001 0.001" />
       </geometry>
     </collision>
@@ -78,12 +82,14 @@
       <origin xyz="-0.383252 -0.383252 -0.076" rpy="0 0 0" />
       <geometry>
-        <mesh filename="package://r26a_urdf/meshes/omni_4_1.stl" scale="0.001 0.001 0.001" />
-      </geometry>
-      <material name="silver" />
-    </visual>
-    <collision>
-      <origin xyz="-0.03335 -0.03335 0" rpy="0 0 0" />
-      <geometry>
-        <sphere radius="0.076" />
+        <mesh filename="file://$(find r26a_urdf)/meshes/omni_4_1.stl"
+          scale="0.001 0.001 0.001" />
+      </geometry>
+      <material name="silver" />
+    </visual>
+    <collision>
+      <origin xyz="-0.383252 -0.383252 -0.076" rpy="0 0 0" />
+      <geometry>
+        <mesh filename="file://$(find r26a_urdf)/meshes/omni_4_1.stl"
+          scale="0.001 0.001 0.001" />
       </geometry>
     </collision>
@@ -98,12 +104,14 @@
       <origin xyz="0.383252 -0.383252 -0.076" rpy="0 0 0" />
       <geometry>
-        <mesh filename="package://r26a_urdf/meshes/omni_3_1.stl" scale="0.001 0.001 0.001" />
-      </geometry>
-      <material name="silver" />
-    </visual>
-    <collision>
-      <origin xyz="0.03335 -0.03335 0" rpy="0 0 0" />
-      <geometry>
-        <sphere radius="0.076" />
+        <mesh filename="file://$(find r26a_urdf)/meshes/omni_3_1.stl"
+          scale="0.001 0.001 0.001" />
+      </geometry>
+      <material name="silver" />
+    </visual>
+    <collision>
+      <origin xyz="0.383252 -0.383252 -0.076" rpy="0 0 0" />
+      <geometry>
+        <mesh filename="file://$(find r26a_urdf)/meshes/omni_3_1.stl"
+          scale="0.001 0.001 0.001" />
       </geometry>
     </collision>
@@ -118,5 +126,6 @@
       <origin xyz="-0.08 0.374382 -0.433095" rpy="0 0 0" />
       <geometry>
-        <mesh filename="package://r26a_urdf/meshes/r_lidar_1.stl" scale="0.001 0.001 0.001" />
+        <mesh filename="file://$(find r26a_urdf)/meshes/r_lidar_1.stl"
+          scale="0.001 0.001 0.001" />
       </geometry>
       <material name="silver" />
@@ -125,5 +134,6 @@
       <origin xyz="-0.08 0.374382 -0.433095" rpy="0 0 0" />
       <geometry>
-        <mesh filename="package://r26a_urdf/meshes/r_lidar_1.stl" scale="0.001 0.001 0.001" />
+        <mesh filename="file://$(find r26a_urdf)/meshes/r_lidar_1.stl"
+          scale="0.001 0.001 0.001" />
       </geometry>
     </collision>
@@ -138,5 +148,6 @@
       <origin xyz="-0.015 0.250446 -0.4402" rpy="0 0 0" />
       <geometry>
-        <mesh filename="package://r26a_urdf/meshes/r_cam_1.stl" scale="0.001 0.001 0.001" />
+        <mesh filename="file://$(find r26a_urdf)/meshes/r_cam_1.stl"
+          scale="0.001 0.001 0.001" />
       </geometry>
       <material name="silver" />
@@ -145,5 +156,6 @@
       <origin xyz="-0.015 0.250446 -0.4402" rpy="0 0 0" />
       <geometry>
-        <mesh filename="package://r26a_urdf/meshes/r_cam_1.stl" scale="0.001 0.001 0.001" />
+        <mesh filename="file://$(find r26a_urdf)/meshes/r_cam_1.stl"
+          scale="0.001 0.001 0.001" />
       </geometry>
     </collision>
@@ -153,10 +165,11 @@
       <origin xyz="-0.029749880192293236 0.009806199358828122 1.596729986563794e-07" rpy="0 0 0" />
       <mass value="0.017157190826827023" />
-      <inertia ixx="1.0e-05" iyy="1.4e-05" izz="1.5e-05" ixy="-0.0" iyz="-0.0" ixz="-0.0" />
+      <inertia ixx="1e-06" iyy="1.4e-05" izz="1.5e-05" ixy="-0.0" iyz="-0.0" ixz="-0.0" />
     </inertial>
     <visual>
       <origin xyz="-0.02975 0.251646 -0.4612" rpy="0 0 0" />
       <geometry>
-        <mesh filename="package://r26a_urdf/meshes/r_cam_body_1.stl" scale="0.001 0.001 0.001" />
+        <mesh filename="file://$(find r26a_urdf)/meshes/r_cam_body_1.stl"
+          scale="0.001 0.001 0.001" />
       </geometry>
       <material name="silver" />
@@ -165,5 +178,6 @@
       <origin xyz="-0.02975 0.251646 -0.4612" rpy="0 0 0" />
       <geometry>
-        <mesh filename="package://r26a_urdf/meshes/r_cam_body_1.stl" scale="0.001 0.001 0.001" />
+        <mesh filename="file://$(find r26a_urdf)/meshes/r_cam_body_1.stl"
+          scale="0.001 0.001 0.001" />
       </geometry>
     </collision>
@@ -178,5 +192,6 @@
       <origin xyz="-0.0 0.333335 -0.394095" rpy="0 0 0" />
       <geometry>
-        <mesh filename="package://r26a_urdf/meshes/r_lidar_head_1.stl" scale="0.001 0.001 0.001" />
+        <mesh filename="file://$(find r26a_urdf)/meshes/r_lidar_head_1.stl"
+          scale="0.001 0.001 0.001" />
       </geometry>
       <material name="silver" />
@@ -185,29 +200,79 @@
       <origin xyz="-0.0 0.333335 -0.394095" rpy="0 0 0" />
       <geometry>
-        <mesh filename="package://r26a_urdf/meshes/r_lidar_head_1.stl" scale="0.001 0.001 0.001" />
-      </geometry>
-    </collision>
-  </link>
-  <gazebo reference="r_lidar_head_1">
-    <material>Gazebo/Blue</material>
-    <sensor type="lidar" name="lidar">
-      <pose>0 0 0 0 0 0</pose>
+        <mesh filename="file://$(find r26a_urdf)/meshes/r_lidar_head_1.stl"
+          scale="0.001 0.001 0.001" />
+      </geometry>
+    </collision>
+  </link>
+  <!-- Gazebo-specific sensor tags are removed here so the URDF/Xacro preview can render the model
+  cleanly. -->
+  <joint name="joint_omni_2" type="continuous">
+    <origin xyz="-0.383252 -0.383252 0.076" rpy="0 0 0" />
+    <parent link="base_link" />
+    <child link="omni_2_1" />
+    <axis xyz="0.707107 0.707107 -0.0" />
+  </joint>
+  <joint name="joint_omni_1" type="continuous">
+    <origin xyz="0.383252 -0.383252 0.076" rpy="0 0 0" />
+    <parent link="base_link" />
+    <child link="omni_1_1" />
+    <axis xyz="-0.707107 0.707107 -0.0" />
+  </joint>
+  <joint name="joint_omni_4" type="continuous">
+    <origin xyz="0.383252 0.383252 0.076" rpy="0 0 0" />
+    <parent link="base_link" />
+    <child link="omni_4_1" />
+    <axis xyz="-0.707107 -0.707107 0.0" />
+  </joint>
+  <joint name="joint_omni_3" type="continuous">
+    <origin xyz="-0.383252 0.383252 0.076" rpy="0 0 0" />
+    <parent link="base_link" />
+    <child link="omni_3_1" />
+    <axis xyz="0.707107 -0.707107 0.0" />
+  </joint>
+  <joint name="joint_lidar" type="fixed">
+    <origin xyz="0.08 -0.374382 0.433095" rpy="-0.5708 0 0" />
+    <parent link="base_link" />
+    <child link="r_lidar_1" />
+    <axis xyz="-1.0 0.0 0.0" />
+  </joint>
+  <joint name="joint_camera" type="fixed">
+    <origin xyz="0.015 -0.250446 0.4402" rpy="0.2 0 0" />
+    <parent link="base_link" />
+    <child link="r_cam_1" />
+    <axis xyz="-1.0 0.0 0.0" />
+  </joint>
+  <joint name="joint_camera_body" type="fixed">
+    <origin xyz="0.01475 -0.0012 0.021" rpy="0 0 0" />
+    <parent link="r_cam_1" />
+    <child link="r_cam_body_1" />
+  </joint>
+  <joint name="joint_lidar_head" type="fixed">
+    <origin xyz="-0.08 0.041047 -0.039" rpy="0 0 0" />
+    <parent link="r_lidar_1" />
+    <child link="r_lidar_head_1" />
+    <axis xyz="0.0 -0.0 -1.0" />
+  </joint>
+<gazebo reference="r_lidar_head_1">
+    <sensor name="lidar" type="gpu_lidar">
+      <pose relative_to="r_lidar_head_1">0 0 0 0 0 0</pose>
+      <always_on>true</always_on>
       <visualize>true</visualize>
-      <update_rate>15</update_rate>
-      <topic>scan</topic>
-      <gz_frame_id>r_lidar_head_1</gz_frame_id>
-      <ray>
+      <update_rate>10</update_rate>
+      <!-- 変更: トピック名を絶対パスにする -->
+      <topic>/scan</topic>
+      <lidar>
         <scan>
           <horizontal>
-            <samples>400</samples>
-            <resolution>1</resolution>
-            <min_angle>-2.35619449</min_angle>
-            <max_angle>2.35619449</max_angle>
+            <samples>360</samples>
+            <resolution>1.0</resolution>
+            <min_angle>-3.14159</min_angle>
+            <max_angle>3.14159</max_angle>
           </horizontal>
         </scan>
         <range>
-          <min>0.05</min>
-          <max>25.0</max>
-          <resolution>0.001</resolution>
+          <min>0.12</min>
+          <max>10.0</max>
+          <resolution>0.01</resolution>
         </range>
         <noise>
@@ -216,53 +281,6 @@
           <stddev>0.01</stddev>
         </noise>
-      </ray>
+      </lidar>
     </sensor>
   </gazebo>
-  <joint name="回転 5" type="continuous">
-    <origin xyz="-0.383252 -0.383252 0.076" rpy="0 0 0" />
-    <parent link="base_link" />
-    <child link="omni_2_1" />
-    <axis xyz="0.707107 0.707107 -0.0" />
-  </joint>
-  <joint name="回転 6" type="continuous">
-    <origin xyz="0.383252 -0.383252 0.076" rpy="0 0 0" />
-    <parent link="base_link" />
-    <child link="omni_1_1" />
-    <axis xyz="-0.707107 0.707107 -0.0" />
-  </joint>
-  <joint name="回転 7" type="continuous">
-    <origin xyz="0.383252 0.383252 0.076" rpy="0 0 0" />
-    <parent link="base_link" />
-    <child link="omni_4_1" />
-    <axis xyz="-0.707107 -0.707107 0.0" />
-  </joint>
-  <joint name="回転 8" type="continuous">
-    <origin xyz="-0.383252 0.383252 0.076" rpy="0 0 0" />
-    <parent link="base_link" />
-    <child link="omni_3_1" />
-    <axis xyz="0.707107 -0.707107 0.0" />
-  </joint>
-  <joint name="回転 9" type="fixed">
-    <origin xyz="0.08 -0.374382 0.433095" rpy="-0.5708 0 0" />
-    <parent link="base_link" />
-    <child link="r_lidar_1" />
-    <axis xyz="-1.0 0.0 0.0" />
-  </joint>
-  <joint name="回転 14" type="fixed">
-    <origin xyz="0.015 -0.250446 0.4402" rpy="0 0 0" />
-    <parent link="base_link" />
-    <child link="r_cam_1" />
-    <axis xyz="-1.0 0.0 0.0" />
-  </joint>
-  <joint name="剛性 15" type="fixed">
-    <origin xyz="0.01475 -0.0012 0.021" rpy="0 0 0" />
-    <parent link="r_cam_1" />
-    <child link="r_cam_body_1" />
-  </joint>
-  <joint name="回転 17" type="continuous">
-    <origin xyz="-0.08 0.041047 -0.039" rpy="0 0 0" />
-    <parent link="r_lidar_1" />
-    <child link="r_lidar_head_1" />
-    <axis xyz="0.0 -0.0 -1.0" />
-  </joint>
 </robot>

Commit message: とりまコミット。urdf変えた。

File: src/r26a_urdf/r26a_urdf.xacro (robot description, xacro)
@@ -207,5 +207,17 @@
   <!-- Gazebo-specific sensor tags are removed here so the URDF/Xacro preview can render the model
   cleanly. -->
+  <joint name="joint_omni_1" type="continuous">
+    <origin xyz="0.383252 0.383252 0.076" rpy="0 0 0" />
+    <parent link="base_link" />
+    <child link="omni_4_1" />
+    <axis xyz="-0.707107 -0.707107 0.0" />
+  </joint>
   <joint name="joint_omni_2" type="continuous">
+    <origin xyz="0.383252 -0.383252 0.076" rpy="0 0 0" />
+    <parent link="base_link" />
+    <child link="omni_1_1" />
+    <axis xyz="-0.707107 0.707107 -0.0" />
+  </joint>
+  <joint name="joint_omni_3" type="continuous">
     <origin xyz="-0.383252 -0.383252 0.076" rpy="0 0 0" />
     <parent link="base_link" />
@@ -213,17 +225,5 @@
     <axis xyz="0.707107 0.707107 -0.0" />
   </joint>
-  <joint name="joint_omni_1" type="continuous">
-    <origin xyz="0.383252 -0.383252 0.076" rpy="0 0 0" />
-    <parent link="base_link" />
-    <child link="omni_1_1" />
-    <axis xyz="-0.707107 0.707107 -0.0" />
-  </joint>
   <joint name="joint_omni_4" type="continuous">
-    <origin xyz="0.383252 0.383252 0.076" rpy="0 0 0" />
-    <parent link="base_link" />
-    <child link="omni_4_1" />
-    <axis xyz="-0.707107 -0.707107 0.0" />
-  </joint>
-  <joint name="joint_omni_3" type="continuous">
     <origin xyz="-0.383252 0.383252 0.076" rpy="0 0 0" />
     <parent link="base_link" />
@@ -259,5 +259,5 @@
       <always_on>true</always_on>
       <visualize>true</visualize>
-      <update_rate>10</update_rate>
+      <update_rate>100</update_rate>
       <!-- 変更: トピック名を絶対パスにする -->
       <topic>/scan</topic>
@@ -265,22 +265,96 @@
         <scan>
           <horizontal>
-            <samples>360</samples>
+            <samples>200</samples>
             <resolution>1.0</resolution>
             <min_angle>-3.14159</min_angle>
             <max_angle>3.14159</max_angle>
           </horizontal>
+          <vertical>
+            <samples>50</samples>
+            <resolution>1.0</resolution>
+            <min_angle>-1.570796</min_angle>
+            <max_angle>0.0</max_angle>
+          </vertical>
         </scan>
         <range>
-          <min>0.12</min>
-          <max>10.0</max>
-          <resolution>0.01</resolution>
+          <min>0.05</min>
+          <max>20.0</max>
+          <resolution>0.0045</resolution>
         </range>
         <noise>
           <type>gaussian</type>
           <mean>0.0</mean>
-          <stddev>0.01</stddev>
+          <stddev>0.02</stddev>
         </noise>
       </lidar>
     </sensor>
   </gazebo>
+  <!-- Wheel Friction settings for smooth Gazebo Omni-wheel sliding -->
+  <gazebo reference="omni_1_1">
+    <mu1>0.8</mu1>
+    <mu2>0.01</mu2>
+    <fdir1>0.707107 0.707107 0</fdir1>
+  </gazebo>
+  <gazebo reference="omni_2_1">
+    <mu1>0.8</mu1>
+    <mu2>0.01</mu2>
+    <fdir1>-0.707107 0.707107 0</fdir1>
+  </gazebo>
+  <gazebo reference="omni_3_1">
+    <mu1>0.8</mu1>
+    <mu2>0.01</mu2>
+    <fdir1>-0.707107 -0.707107 0</fdir1>
+  </gazebo>
+  <gazebo reference="omni_4_1">
+    <mu1>0.8</mu1>
+    <mu2>0.01</mu2>
+    <fdir1>0.707107 -0.707107 0</fdir1>
+  </gazebo>
+  <!-- Gazebo Harmonic Plugins -->
+  <gazebo>
+    <!-- Joint Controllers for individual wheel velocity control -->
+    <plugin
+      filename="gz-sim-joint-controller-system"
+      name="gz::sim::systems::JointController">
+      <joint_name>joint_omni_1</joint_name>
+      <topic>/omni_1/cmd_vel</topic>
+      <sub_topic>cmd_vel</sub_topic>
+    </plugin>
+    <plugin
+      filename="gz-sim-joint-controller-system"
+      name="gz::sim::systems::JointController">
+      <joint_name>joint_omni_2</joint_name>
+      <topic>/omni_2/cmd_vel</topic>
+      <sub_topic>cmd_vel</sub_topic>
+    </plugin>
+    <plugin
+      filename="gz-sim-joint-controller-system"
+      name="gz::sim::systems::JointController">
+      <joint_name>joint_omni_3</joint_name>
+      <topic>/omni_3/cmd_vel</topic>
+      <sub_topic>cmd_vel</sub_topic>
+    </plugin>
+    <plugin
+      filename="gz-sim-joint-controller-system"
+      name="gz::sim::systems::JointController">
+      <joint_name>joint_omni_4</joint_name>
+      <topic>/omni_4/cmd_vel</topic>
+      <sub_topic>cmd_vel</sub_topic>
+    </plugin>
+    <!-- Joint State Publisher Plugin -->
+    <plugin
+      filename="gz-sim-joint-state-publisher-system"
+      name="gz::sim::systems::JointStatePublisher">
+      <topic>/joint_states</topic>
+    </plugin>
+    <!-- Odometry Publisher Plugin for Field-Oriented Control -->
+    <plugin
+      filename="gz-sim-odometry-publisher-system"
+      name="gz::sim::systems::OdometryPublisher">
+      <odom_topic>/odom</odom_topic>
+      <tf_topic>/tf</tf_topic>
+      <odom_frame>odom</odom_frame>
+      <robot_base_frame>base_link</robot_base_frame>
+    </plugin>
+  </gazebo>
 </robot>
